Commit message: Introduce parameters for the leg joints for the calibration offsets.

File: nao_description/urdf/calibration_joint_offsets.xacro (robot description, xacro)
@@ -1,4 +1,5 @@
 <?xml version="1.0"?>
 <robot>
+<!-- head joint offsets -->
 <property name="HeadPitch_p" value="0" />
 <property name="HeadPitch_r" value="0" />
@@ -7,4 +8,5 @@
 <property name="HeadYaw_r" value="0" />
 <property name="HeadYaw_y" value="0" />
+<!-- left arm joint offsets -->
 <property name="LElbowRoll_p" value="0" />
 <property name="LElbowRoll_r" value="0" />
@@ -19,4 +21,5 @@
 <property name="LShoulderRoll_r" value="0" />
 <property name="LShoulderRoll_y" value="0" />
+<!-- right arm joint offsets -->
 <property name="RElbowRoll_p" value="0" />
 <property name="RElbowRoll_r" value="0" />
@@ -31,3 +34,35 @@
 <property name="RShoulderRoll_r" value="0" />
 <property name="RShoulderRoll_y" value="0" />
+<!-- left leg joint offsets -->
+<property name="LHipYawPitch_r" value="0" />
+<property name="LHipYawPitch_p" value="0" />
+<property name="LHipYawPitch_y" value="0" />
+<property name="LHipPitch_r" value="0" />
+<property name="LHipPitch_p" value="0" />
+<property name="LHipPitch_y" value="0" />
+<property name="LKneePitch_r" value="0" />
+<property name="LKneePitch_p" value="0" />
+<property name="LKneePitch_y" value="0" />
+<property name="LAnklePitch_r" value="0" />
+<property name="LAnklePitch_p" value="0" />
+<property name="LAnklePitch_y" value="0" />
+<property name="LHipRoll_r" value="0" />
+<property name="LHipRoll_p" value="0" />
+<property name="LHipRoll_y" value="0" />
+<!-- left leg joint offsets -->
+<property name="RHipYawPitch_r" value="0" />
+<property name="RHipYawPitch_p" value="0" />
+<property name="RHipYawPitch_y" value="0" />
+<property name="RHipPitch_r" value="0" />
+<property name="RHipPitch_p" value="0" />
+<property name="RHipPitch_y" value="0" />
+<property name="RKneePitch_r" value="0" />
+<property name="RKneePitch_p" value="0" />
+<property name="RKneePitch_y" value="0" />
+<property name="RAnklePitch_r" value="0" />
+<property name="RAnklePitch_p" value="0" />
+<property name="RAnklePitch_y" value="0" />
+<property name="RHipRoll_r" value="0" />
+<property name="RHipRoll_p" value="0" />
+<property name="RHipRoll_y" value="0" />
 </robot>

File: nao_description/urdf/nao_robot_v4_structure.urdf.xacro (robot description, xacro)
@@ -297,5 +297,5 @@
     <parent link="torso"/>
     <child link="LHipYawPitch_link"/>
-    <origin xyz="0 0.05 -0.085" rpy="0 0 0"/>
+    <origin xyz="0 0.05 -0.085" rpy="0 ${LHipYawPitch_p} ${LHipYawPitch_y}"/>
     <axis xyz="0 0.707106 -0.707106"/>
     <limit velocity="3.0" effort="30" lower="-1.145303" upper="0.740810"/>
@@ -304,14 +304,14 @@
     <parent link="torso"/>
     <child link="RHipYawPitch_link"/>
-    <origin xyz="0 -0.05 -0.085" rpy="0 0 0"/>
+    <origin xyz="0 -0.05 -0.085" rpy="0 ${RHipYawPitch_p} ${RHipYawPitch_y}"/>
     <axis xyz="0 0.707106 0.707106"/>
     <limit velocity="3.0" effort="30" lower="-1.145303" upper="0.740810"/>
     <mimic joint="LHipYawPitch" multiplier="1" offset="0"/>
   </joint>
-  <xacro:macro name="leg_joints" params="side reflect">
+  <xacro:macro name="leg_joints" params="side reflect HipPitch_p KneePitch_p AnklePitch_p">
   <joint name="${side}HipPitch" type="revolute">
     <parent link="${side}HipRoll_link"/>
     <child link="${side}HipPitch_link"/>
-    <origin xyz="0 0 0" rpy="0 0 0"/>
+    <origin xyz="0 0 0" rpy="0 ${HipPitch_p} 0"/>
     <axis xyz="0 1 0"/>
     <!--Nao V3 and V4-->
@@ -323,5 +323,5 @@
     <parent link="${side}HipPitch_link"/>
     <child link="${side}KneePitch_link"/>
-    <origin xyz="0 0 -0.1" rpy="0 0 0"/>
+    <origin xyz="0 0 -0.1" rpy="0 ${KneePitch_p} 0"/>
     <axis xyz="0 1 0"/>
     <!-- LKneePitch limits: -0.092346 .. 2.112528 -->
@@ -332,5 +332,5 @@
     <parent link="${side}KneePitch_link"/>
     <child link="${side}AnklePitch_link"/>
-    <origin xyz="0 0 -0.10290" rpy="0 0 0"/>
+    <origin xyz="0 0 -0.10290" rpy="0 ${AnklePitch_p} 0"/>
     <axis xyz="0 1 0"/>
     <!-- LAnklePitch limits: -1.189516 .. 0.922747 -->
@@ -342,5 +342,5 @@
     <parent link="LHipYawPitch_link"/>
     <child link="LHipRoll_link"/>
-    <origin xyz="0 0 0" rpy="0 0 0"/>
+    <origin xyz="0 0 0" rpy="${LHipRoll_r} 0 0"/>
     <axis xyz="1 0 0"/>
     <limit velocity="3.0" effort="30" lower="-0.379472" upper="0.790477"/>
@@ -349,5 +349,5 @@
     <parent link="RHipYawPitch_link"/>
     <child link="RHipRoll_link"/>
-    <origin xyz="0 0 0" rpy="0 0 0"/>
+    <origin xyz="0 0 0" rpy="${RHipRoll_r} 0 0"/>
     <axis xyz="1 0 0"/>
     <limit velocity="3.0" effort="30" lower="-0.738321" upper="0.414754"/>
@@ -387,5 +387,5 @@
     <origin xyz="0 0 -0.04519" />
   </joint>
-  <xacro:leg_joints side="L" reflect="-1"/>
-  <xacro:leg_joints side="R" reflect="1"/>
+  <xacro:leg_joints side="L" reflect="-1" HipPitch_p="${LHipPitch_p}" KneePitch_p="${LKneePitch_p}" AnklePitch_p="${LAnklePitch_p}" />
+  <xacro:leg_joints side="R" reflect="1" HipPitch_p="${RHipPitch_p}" KneePitch_p="${RKneePitch_p}" AnklePitch_p="${RAnklePitch_p}" />
 </robot>
